File: kicad/esp485/esp485.kicad_pcb (KiCad board)
At the start: 2 copper layers, 0 parts

Commit message: donw some work
Parts:
- added C1: CP, Capacitors_THT:CP_Radial_D6.3mm_P2.50mm, F.Cu at (128.0, 105.3)
- added J1: Conn_01x04, Pin_Headers:Pin_Header_Straight_1x04_Pitch2.54mm, F.Cu at (121.9, 104.1)
- added J2: Conn_02x06_Odd_Even, Pin_Headers:Pin_Header_Straight_2x06_Pitch2.54mm, F.Cu at (157.5, 94.0)
- added R1: 10K, Resistors_SMD:R_0805_HandSoldering, B.Cu at (137.8, 98.6)
- added R10: 100, Resistors_SMD:R_0805_HandSoldering, F.Cu at (125.7, 94.0)
- added R2: 10K, Resistors_SMD:R_0805_HandSoldering, B.Cu at (142.4, 98.6)
- added R3: 10K, Resistors_SMD:R_0805_HandSoldering, B.Cu at (140.1, 98.6)
- added R4: 20K, Resistors_SMD:R_0805_HandSoldering, F.Cu at (130.8, 94.0)
- added R5: 20K, Resistors_SMD:R_0805_HandSoldering, F.Cu at (128.3, 94.0)
- added R7: 10K, Resistors_SMD:R_0805_HandSoldering, B.Cu at (147.2, 98.6)
- added R8: 10K, Resistors_SMD:R_0805_HandSoldering, B.Cu at (144.9, 98.6)
- added R9: 10K, Resistors_SMD:R_0805_HandSoldering, B.Cu at (147.7, 105.5)
- added U1: MAX3485, Housings_SOIC:SOIC-8_3.9x4.9mm_Pitch1.27mm, F.Cu at (128.3, 100.3)
- added U2: ESP-WROOM-02, ESP8266:ESP-13-WROOM-02, F.Cu at (134.0, 97.2)
Routing:
- net GND: track 0.00 -> 79.1 mm, vias 0 -> 2
- net +3V3: track 0.00 -> 69.0 mm, vias 0 -> 1
- net Net-(J2-Pad9): track 0.00 -> 47.9 mm, vias 0 -> 2
- net Net-(J2-Pad8): track 0.00 -> 38.9 mm, vias 0 -> 3
- net Net-(J2-Pad6): track 0.00 -> 31.8 mm, vias 0 -> 1
- net Net-(J2-Pad4): track 0.00 -> 28.6 mm, vias 0 -> 1
- net Net-(R8-Pad2): track 0.00 -> 28.4 mm, vias 0 -> 2
- net Net-(J2-Pad10): track 0.00 -> 27.2 mm, vias 0 -> 1
- net Net-(J2-Pad2): track 0.00 -> 24.4 mm, vias 0 -> 1
- net Net-(J1-Pad3): track 0.00 -> 19.9 mm, vias 0 -> 1
- net Net-(J2-Pad7): track 0.00 -> 18.9 mm
- net Net-(R2-Pad1): track 0.00 -> 17.4 mm, vias 0 -> 1
- net Net-(J2-Pad1): track 0.00 -> 16.9 mm
- net Net-(J2-Pad3): track 0.00 -> 14.6 mm
- net Net-(J1-Pad2): track 0.00 -> 13.8 mm
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Other:
- board outline added: 43.2 x 20.3 mm
- net class Default: via_dia 0.6 -> 0.8
- rule via_min_size: 0.4 -> 0.8
