File: kicad/esp485-base/esp485-base.kicad_pcb (KiCad board)
At the start: 2 copper layers, 48.3 x 20.3 mm, 7 parts, among them J1 Conn_01x04, J2 Conn_02x06_Odd_Even, J3 Conn_01x07, J4 Conn_01x07, J5 Conn_01x03, U1 AMS1117-3.3

Commit message: stop using modules from github to enable 3d models
Parts:
- J1: footprint Pin_Headers:Pin_Header_Straight_1x04_Pitch2.54mm -> Connector_PinHeader_2.54mm:PinHeader_1x04_P2.54mm_Vertical; moved to B.Cu
- J2: footprint Pin_Headers:Pin_Header_Straight_2x06_Pitch2.54mm -> Connector_PinHeader_2.54mm:PinHeader_2x06_P2.54mm_Vertical; moved to B.Cu
- J3, J4: footprint Pin_Headers:Pin_Header_Straight_1x07_Pitch2.54mm -> Connector_PinSocket_2.54mm:PinSocket_1x07_P2.54mm_Vertical
- J5: footprint Pin_Headers:Pin_Header_Straight_1x03_Pitch2.54mm -> Connector_PinHeader_2.54mm:PinHeader_1x03_P2.54mm_Vertical
- U1: footprint TO_SOT_Packages_SMD:SOT-223-3_TabPin2 -> Package_TO_SOT_SMD:SOT-223-3_TabPin2
- moved J2 2.54 mm to (160.0, 94.0), turned to 180 degrees
- turned J1 to 0 degrees
Connections:
- J2 pad 1: Net-(J2-Pad1) -> GND
- J2 pad 2: GND -> Net-(J2-Pad2)
- J3 pad 1: Net-(J2-Pad1) -> Net-(J2-Pad2)
- J3 pad 2: Net-(J2-Pad3) -> Net-(J2-Pad4)
- J3 pad 3: Net-(J2-Pad5) -> Net-(J2-Pad6)
- J3 pad 4: Net-(J2-Pad7) -> Net-(J2-Pad8)
- J3 pad 5: Net-(J2-Pad9) -> Net-(J2-Pad10)
- J4 pad 2: Net-(J2-Pad8) -> Net-(J2-Pad7)
- J4 pad 3: Net-(J2-Pad11) -> Net-(J2-Pad12)
- J4 pad 4: Net-(J2-Pad10) -> Net-(J2-Pad9)
- J4 pad 5: Net-(J2-Pad4) -> Net-(J2-Pad3)
- J4 pad 6: Net-(J2-Pad6) -> Net-(J2-Pad5)
- J4 pad 7: Net-(J2-Pad12) -> Net-(J2-Pad11)
- J5 pad 1: Net-(J2-Pad11) -> Net-(J2-Pad12)
- J5 pad 2: Net-(J2-Pad8) -> Net-(J2-Pad7)
- U1 pad 2: Net-(J2-Pad1) -> Net-(J2-Pad2)
Routing:
- net Net-(J2-Pad2): track 0.00 -> 36.3 mm
- net Net-(J2-Pad1): track 36.3 -> 0.00 mm
- net Net-(J2-Pad4): track 10.2 -> 33.0 mm
- net Net-(J2-Pad3): track 33.0 -> 10.2 mm
- net Net-(J2-Pad9): track 25.9 -> 6.93 mm
- net Net-(J2-Pad10): track 6.93 -> 25.9 mm
- net Net-(J2-Pad6): track 12.7 -> 30.6 mm
- net Net-(J2-Pad5): track 30.6 -> 12.7 mm
- net Net-(J2-Pad12): track 5.61 -> 23.1 mm
- net Net-(J2-Pad11): track 23.1 -> 5.61 mm
- net Net-(J2-Pad8): track 21.7 -> 31.8 mm
- net Net-(J2-Pad7): track 31.8 -> 21.7 mm
- net GND: track 71.0 -> 72.2 mm
