File: kicad/usbesp/usbesp.kicad_pcb (KiCad board)
At the start: 2 copper layers, 16.5 x 13.6 mm, 11 parts, among them J1 USB_B_Micro, J2 Conn_01x06, J3 Conn_01x06, Q1 S9013, Q2 S9013, U1 FT232RL

Commit message: schematic was wrong
Parts:
- moved R1 5.63 mm to (147.7, 101.5), turned to 270 degrees
- moved R2 3.26 mm to (154.3, 101.3), turned to 90 degrees
- moved Q1 2.09 mm to (150.7, 103.0)
- moved Q2 2.07 mm to (150.7, 99.4)
Connections:
- J1 pad 4: Net-(J1-Pad4) -> (no net)
- Q1 pad 2: Net-(Q1-Pad2) -> /DTR
- Q2 pad 1: Net-(Q1-Pad2) -> Net-(Q2-Pad1)
- Q2 pad 2: Net-(Q1-Pad1) -> /RTS
- R2 pad 2: Net-(Q1-Pad2) -> Net-(Q2-Pad1)
- U1 pad 10: Net-(U1-Pad10) -> (no net)
- U1 pad 11: Net-(U1-Pad11) -> (no net)
- U1 pad 12: Net-(U1-Pad12) -> (no net)
- U1 pad 13: Net-(U1-Pad13) -> (no net)
- U1 pad 14: Net-(U1-Pad14) -> (no net)
- U1 pad 19: Net-(U1-Pad19) -> (no net)
- U1 pad 22: Net-(U1-Pad22) -> (no net)
- U1 pad 23: Net-(U1-Pad23) -> (no net)
- U1 pad 27: Net-(U1-Pad27) -> (no net)
- U1 pad 28: Net-(U1-Pad28) -> (no net)
- U1 pad 6: Net-(U1-Pad6) -> (no net)
- U1 pad 9: Net-(U1-Pad9) -> (no net)
Routing:
- net /3v3: track 33.3 -> 22.9 mm
- net Net-(Q1-Pad2): track 8.38 -> 0.00 mm
- net Net-(Q1-Pad1): track 6.57 -> 2.24 mm
- net /RTS: track 8.42 -> 11.7 mm
- net GND: track 19.0 -> 22.1 mm, vias 2 -> 3
- net Net-(Q2-Pad1): track 0.00 -> 2.62 mm
- net /RESET: track 9.74 -> 7.28 mm
- net /IO0: track 4.09 -> 6.03 mm
- net /DTR: track 11.9 -> 10.5 mm
- net /VBUS: track 29.8 -> 29.0 mm, vias 0 -> 1
- net /USBDP: track 10.6 -> 11.2 mm
Other:
- board size 16.5 x 13.6 mm -> 15.2 x 12.7 mm
