File: kicad/esp485-32/esp485-32.kicad_pcb (KiCad board)
At the start: 4 copper layers, 25.4 x 25.4 mm, 16 parts, among them J1 Conn_01x08, J2 Conn_01x08, U1 MAX3485, U2 ESP32-WROOM, U3 ADP3338-3.3

Commit message: esp485-32 done
Parts:
- removed C4: C, Capacitor_SMD:C_1206_3216Metric_Pad1.42x1.75mm_HandSolder
- removed R10: 100, Resistor_SMD:R_0805_2012Metric_Pad1.15x1.40mm_HandSolder
- removed R2: 10K, Resistor_SMD:R_0603_1608Metric_Pad1.05x0.95mm_HandSolder
- moved C5 10.8 mm to (144.4, 106.8), turned to 270 degrees
- moved R1 10.7 mm to (145.4, 103.3), turned to 90 degrees
- moved C2 9.96 mm to (137.4, 106.7)
- moved C1 9.86 mm to (139.7, 106.7)
- moved C3 9.86 mm to (142.2, 106.7)
- moved R8 5.48 mm to (141.2, 112.9)
- moved U1 5.48 mm to (140.8, 112.9)
- moved R4 5.08 mm to (134.1, 112.4)
- moved R5 5.01 mm to (134.1, 114.6)
Routing:
- net +3V3: track 3.83 -> 53.5 mm, vias 0 -> 4
- net MISO: track 0.00 -> 30.0 mm, vias 0 -> 1
- net RST: track 3.16 -> 32.5 mm, vias 0 -> 3
- net SCK: track 0.00 -> 29.0 mm, vias 0 -> 1
- net GND: track 25.9 -> 0.00 mm, vias 0 -> 6
- net TOUT: track 0.00 -> 23.7 mm, vias 0 -> 1
- net MOSI: track 0.00 -> 23.1 mm, vias 0 -> 1
- net SS: track 0.00 -> 22.1 mm, vias 0 -> 1
- net IO0: track 10.3 -> 28.8 mm, vias 0 -> 1
- net SDA: track 0.00 -> 17.0 mm, vias 0 -> 1
- net RXD: track 0.00 -> 14.4 mm, vias 0 -> 1
- net TXD: track 0.00 -> 13.7 mm, vias 0 -> 1
- net SCL: track 0.00 -> 11.0 mm, vias 0 -> 1
- net A: track 22.1 -> 15.3 mm
- net B: track 15.3 -> 9.66 mm
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- added copper zone on B.Cu, net GND
- removed copper zone on B.Cu, net +3V3
Other:
- board size 25.4 x 25.4 mm -> 25.4 x 26.7 mm
- copper layers 4 -> 2
- board text added: "3V3"
- board text added: "A/IO2"
- board text added: "B"
- board text added: "GND"
- board text added: "IO0"
- board text added: "MISO"
- board text added: "MOSI"
- board text added: "RST"
- board text added: "RXD"
- board text added: "SCK"
- board text added: "SCL"
- board text added: "SDA"
- board text added: "SS"
- board text added: "TOUT"
- board text added: "TXD"
- board text added: "VIN"
