File: kicad/esp485-13-breakout/esp485-13-breakout.kicad_pcb (KiCad board)
At the start: 2 copper layers, 25.4 x 25.4 mm, 21 parts, among them J1 Conn_01x08, J2 Conn_01x08, SW1 SW_Push, SW2 SW_Push, U1 MAX3485, U2 ESP-WROOM-02, U3 AMS1117-3.3

Commit message: wake resister silk corrected from 1k to 470
Other:
- board text added: "WAKE 470"
- board text removed: "WAKE 1K"
Changed lines of the file:
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@@
     (effects (font (size 0.8 0.8) (thickness 0.14)))
   )
-  (gr_text "WAKE 1K" (at 146.685 112.649) (layer B.SilkS)
+  (gr_text "WAKE 470" (at 146.685 112.649) (layer B.SilkS)
     (effects (font (size 0.6 0.6) (thickness 0.1)) (justify mirror))
   )
