File: kicad/epsolar-junction/epsolar-junction.kicad_pcb (KiCad board)
At the start: 2 copper layers, 87.6 x 50.8 mm, 22 parts, among them J1 Conn_01x02, J10 EDG, J11 DISPLAY, J12 I2C, J13 USB_B_Micro, J14 USBSERIAL, J2 Conn_01x02, J3 Conn_01x02, J4 Conn_01x02, J5 Conn_01x02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

Commit message: terminal block direction corrected
Parts:
- moved J1 11.4 mm to (144.8, 96.5), turned to 180 degrees
- moved J2 11.4 mm to (134.6, 124.5), turned to 0 degrees
Connections:
- J1 pad 1: /LOADPLUS -> GND
- J1 pad 2: GND -> /LOADPLUS
Routing:
- net /LOADPLUS: track 58.1 -> 50.9 mm
- net /A: track 35.8 -> 39.4 mm
- net /B: track 34.4 -> 36.9 mm
